File: kicad_projects/commander/commander.kicad_pcb (KiCad board)
At the start: 2 copper layers, 56 x 100 mm, 18 parts, among them J1 right input IDC14, J10 522710469, J2 left input IDC14, J8 debug out, J9 522710469, Q1 MMFTP3401, SW1 RESET_SWITCH, SW2 SW_Push, SW3 SW_Push, SW4 SW_Push, U1 Pico

Commit message: commander board rev2, pre-manufacture
Parts:
- removed the HOLE_M3 at (158.5, 117.3)
- removed the HOLE_M3 at (111.5, 136.9)
- added HOLE_M3: H2, revolt_footprints:HOLE_M3, F.Cu at (111.5, 119.1)
- added HOLE_M3: H2, revolt_footprints:HOLE_M3, F.Cu at (158.5, 136.4)
- added J11: Conn_02x01, Connector_PinHeader_2.54mm:PinHeader_2x01_P2.54mm_Vertical, B.Cu at (151.6, 125.5)
- added J12: Conn_02x01, Connector_PinHeader_2.54mm:PinHeader_2x01_P2.54mm_Vertical, B.Cu at (153.2, 121.4)
- added J13: Conn_02x01, Connector_PinHeader_2.54mm:PinHeader_2x01_P2.54mm_Vertical, B.Cu at (151.6, 117.3)
- added JP2: SolderJumper_2_Bridged, Jumper:SolderJumper-2_P1.3mm_Bridged2Bar_RoundedPad1.0x1.5mm, B.Cu at (134.6, 132.1)
- added JP3: SolderJumper_2_Bridged, Jumper:SolderJumper-2_P1.3mm_Bridged2Bar_RoundedPad1.0x1.5mm, B.Cu at (129.5, 129.3)
- added JP4: SolderJumper_2_Bridged, Jumper:SolderJumper-2_P1.3mm_Bridged2Bar_RoundedPad1.0x1.5mm, B.Cu at (134.6, 124.2)
- added JP5: SolderJumper_2_Bridged, Jumper:SolderJumper-2_P1.3mm_Bridged2Bar_RoundedPad1.0x1.5mm, B.Cu at (129.5, 121.9)
- added PSP_JOY: PSP1000_JOY, revolt_footprints:PSP1000_JOY, F.Cu at (119.7, 129.2)
- added Q2: NPN - MMBT2222A, Package_TO_SOT_SMD:SOT-23, B.Cu at (151.4, 110.5)
- J10: value 522710469 -> Conn_02x01; footprint revolt_footprints:CON_522710469_MOL -> Connector_PinHeader_2.54mm:PinHeader_2x01_P2.54mm_Vertical; moved to B.Cu
- J9: footprint revolt_footprints:CON_522710469_MOL -> revolt_footprints:HC-FPC-05-09-4RLTAG; moved to B.Cu
- JP1, R2: moved to B.Cu
- Q1: value MMFTP3401 -> AO3401A; moved to B.Cu
- R1: value 220R -> 1k; moved to B.Cu
- SW2, SW3, SW4: footprint revolt_footprints:SW_PG1350_reversible_with_keycap_outline -> keyswitches:Kailh_socket_PG1350_optional
- moved J10 34.0 mm to (153.2, 129.5), turned to 180 degrees
- moved J9 29.0 mm to (122.6, 130.7), turned to 90 degrees
- moved Q1 3.64 mm to (158.5, 112.5), turned to 0 degrees
- moved R2 3.59 mm to (154.7, 112.5)
- moved JP1 2.90 mm to (158.2, 108.5), turned to 0 degrees
- moved R1 2.84 mm to (150.4, 106.4)
- turned SW2 to 0 degrees
Connections:
- net /NOT_LED_ENABLE renamed /LED_ENABLE
- J10 pad 1: unconnected-(J10-Pad1) -> GND
- J10 pad 2: unconnected-(J10-Pad2) -> Net-(J10-Pin_2)
- J9 pad 1: unconnected-(J9-Pad1) -> Net-(J10-Pin_2)
- J9 pad 2: unconnected-(J9-Pad2) -> Net-(J11-Pin_2)
- J9 pad 3: unconnected-(J9-Pad3) -> Net-(J12-Pin_2)
- J9 pad 4: unconnected-(J9-Pad4) -> Net-(J13-Pin_2)
- R1 pad 1: Net-(Q1-G) -> Net-(Q2-B)
- R2 pad 1: 5V -> Net-(Q1-G)
- R2 pad 2: Net-(Q1-G) -> 5V
- SW2 pad 1: unconnected-(SW2-Pad1) -> /LMB
- SW2 pad 2: unconnected-(SW2-Pad2) -> GND
- SW3 pad 1: unconnected-(SW3-Pad1) -> /MMB
- SW3 pad 2: unconnected-(SW3-Pad2) -> GND
- SW4 pad 1: unconnected-(SW4-Pad1) -> /RMB
- SW4 pad 2: unconnected-(SW4-Pad2) -> GND
- U1 pad 19: unconnected-(U1-GPIO14-Pad19) -> /LMB
- U1 pad 20: unconnected-(U1-GPIO15-Pad20) -> /MMB
- U1 pad 6: unconnected-(U1-GPIO4-Pad6) -> /RMB
Routing:
- net /RMB: track 0.00 -> 99.8 mm
- net 3V3: track 0.00 -> 82.0 mm, vias 0 -> 2
- net /X1: track 0.00 -> 74.8 mm, vias 0 -> 1
- net /LMB: track 0.00 -> 74.5 mm
- net /X2: track 0.00 -> 70.9 mm
- net /MMB: track 0.00 -> 51.2 mm
- net Net-(J13-Pin_2): track 0.00 -> 34.5 mm
- net Net-(J12-Pin_2): track 0.00 -> 31.9 mm
- net Net-(J10-Pin_2): track 0.00 -> 30.1 mm
- net Net-(J11-Pin_2): track 0.00 -> 28.7 mm
- net 5V: track 73.0 -> 68.4 mm, vias 1 -> 0
- net /LED_ENABLE: track 45.7 -> 42.7 mm, vias 1 -> 0
- net Net-(Q2-B): track 0.00 -> 2.15 mm
- net LED_5V: track 75.5 -> 76.8 mm
- net /COL1: track 34.9 -> 36.1 mm
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Other:
- board text added: "commander board rev2"
- board text removed: "commander rev2"

Commit message: commander rev2 production files
Parts:
- J9: value 522710469 -> HC-FPC-05-09-4RLTAG
Changed lines of the file:
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@@
 		(tags "kailh,choc")
 		(property "Reference" "SW2"
-			(at 0 -8.255 360)
+			(at 0 -8.255 0)
 			(layer "F.SilkS")
 			(hide yes)
@@
 		)
 		(property "Value" "SW_Push"
-			(at 0 8.25 360)
+			(at 0 8.25 0)
 			(layer "F.Fab")
 			(effects
@@
 		)
 		(property "Footprint" "keyswitches:Kailh_socket_PG1350_optional"
-			(at 0 0 360)
+			(at 0 0 0)
 			(layer "F.Fab")
 			(hide yes)
@@
 		)
 		(property "Datasheet" ""
-			(at 0 0 360)
+			(at 0 0 0)
 			(layer "F.Fab")
 			(hide yes)
@@
 		)
 		(property "Description" "Push button switch, generic, two pins"
-			(at 0 0 360)
+			(at 0 0 0)
 			(layer "F.Fab")
 			(hide yes)
@@
 		)
 		(fp_text user "${REFERENCE}"
-			(at 4.445 -7.62 360)
+			(at 4.445 -7.62 0)
 			(layer "B.SilkS")
 			(effects
@@
 		)
 		(fp_text user "${VALUE}"
-			(at 2.54 -0.635 360)
+			(at 2.54 -0.635 0)
 			(layer "B.Fab")
 			(effects
@@
 		)
 		(fp_text user "${REFERENCE}"
-			(at 3 -5 360)
+			(at 3 -5 0)
 			(layer "B.Fab")
 			(effects
@@
 		)
 		(fp_text user "${REFERENCE}"
-			(at 0 0 360)
+			(at 0 0 0)
 			(layer "F.Fab")
 			(effects
@@
 		(tags "net tie solder jumper bridged")
 		(property "Reference" "JP3"
-			(at 0 1.8 360)
+			(at 0 1.8 0)
 			(layer "B.SilkS")
 			(effects
@@
 		)
 		(property "Value" "SolderJumper_2_Bridged"
-			(at 0 -1.9 360)
+			(at 0 -1.9 0)
 			(layer "B.Fab")
 			(effects
@@
 			)
 		)
+		(property "LCSC" "C17513"
+			(at 0 0 90)
+			(unlocked yes)
+			(layer "B.Fab")
+			(hide yes)
+			(effects
+				(font
+					(size 1 1)
+					(thickness 0.15)
+				)
+				(justify mirror)
+			)
+		)
 		(property ki_fp_filters "R_*")
 		(sheetname "Root")
@@
 			)
 		)
+		(property "LCSC" "C17414"
+			(at 0 0 90)
+			(unlocked yes)
+			(layer "B.Fab")
+			(hide yes)
+			(effects
+				(font
+					(size 1 1)
+					(thickness 0.15)
+				)
+				(justify mirror)
+			)
+		)
 		(property ki_fp_filters "R_*")
 		(sheetname "Root")
@@
 		(tags "net tie solder jumper bridged")
 		(property "Reference" "JP2"
-			(at 0 1.8 360)
+			(at 0 1.8 0)
 			(layer "B.SilkS")
 			(effects
@@
 		)
 		(property "Value" "SolderJumper_2_Bridged"
-			(at 0 -1.9 360)
+			(at 0 -1.9 0)
 			(layer "B.Fab")
 			(effects
@@
 		(tags "Through hole pin header THT 2x01 2.54mm double row")
 		(property "Reference" "J13"
-			(at -3.297 0 360)
+			(at -3.297 0 0)
 			(layer "B.SilkS")
 			(effects
@@
 		)
 		(property "Value" "Conn_02x01"
-			(at 1.27 -2.33 360)
+			(at 1.27 -2.33 0)
 			(layer "B.Fab")
 			(effects
@@
 		(tags "Through hole pin header THT 2x01 2.54mm double row")
 		(property "Reference" "J11"
-			(at -3.297 0 360)
+			(at -3.297 0 0)
 			(layer "B.SilkS")
 			(effects
@@
 		)
 		(property "Value" "Conn_02x01"
-			(at 1.27 -2.33 360)
+			(at 1.27 -2.33 0)
 			(layer "B.Fab")
 			(effects
@@
 		(tags "net tie solder jumper bridged")
 		(property "Reference" "JP5"
-			(at 0 1.8 360)
+			(at 0 1.8 0)
 			(layer "B.SilkS")
 			(effects
@@
 		)
 		(property "Value" "SolderJumper_2_Bridged"
-			(at 0 -1.9 360)
+			(at 0 -1.9 0)
 			(layer "B.Fab")
 			(effects
@@
 		(tags "Through hole pin header THT 2x01 2.54mm double row")
 		(property "Reference" "J12"
-			(at 5.847 0 360)
+			(at 5.847 0 0)
 			(layer "B.SilkS")
 			(effects
@@
 		)
 		(property "Value" "Conn_02x01"
-			(at 1.27 -2.33 360)
+			(at 1.27 -2.33 0)
 			(layer "B.Fab")
 			(effects
@@
 		(sheetfile "commander.kicad_sch")
 		(zone_connect 1)
+		(attr exclude_from_bom)
 		(fp_line
 			(start -1.4 0.3)
@@
 		(tags "Through hole pin header THT 2x01 2.54mm double row")
 		(property "Reference" "J10"
-			(at 5.847 0 360)
+			(at 5.847 0 0)
 			(layer "B.SilkS")
 			(effects
@@
 		)
 		(property "Value" "Conn_02x01"
-			(at 1.27 -2.33 360)
+			(at 1.27 -2.33 0)
 			(layer "B.Fab")
 			(effects
@@
 			)
 		)
-		(property "Value" "522710469"
+		(property "Value" "HC-FPC-05-09-4RLTAG"
 			(at 0 2.8 -90)
 			(unlocked yes)
@@
 			)
 		)
-		(property "Datasheet" "522710469"
+		(property "Datasheet" "HC-FPC-05-09-4RLTAG"
 			(at 0 3.8 -90)
 			(unlocked yes)
@@
 			)
 		)
+		(property "LCSC" "C5213746"
+			(at 0 0 90)
+			(unlocked yes)
+			(layer "B.Fab")
+			(hide yes)
+			(effects
+				(font
+					(size 1 1)
+					(thickness 0.15)
+				)
+				(justify mirror)
+			)
+		)
 		(property ki_fp_filters "CON_522710469_MOL")
 		(sheetname "Root")
@@
 		(tags "net tie solder jumper bridged")
 		(property "Reference" "JP4"
-			(at 0 1.8 360)
+			(at 0 1.8 0)
 			(layer "B.SilkS")
 			(effects
@@
 		)
 		(property "Value" "SolderJumper_2_Bridged"
-			(at 0 -1.9 360)
+			(at 0 -1.9 0)
 			(layer "B.Fab")
 			(effects

Commit message: Correct Column net names
Connections:
- J1 pad 11: /COL4 -> /COL9
- J1 pad 13: /COL5 -> /COL8
- J1 pad 14: /COL6 -> /COL7
- J1 pad 3: /COL0 -> /COL13
- J1 pad 5: /COL1 -> /COL12
- J1 pad 7: /COL2 -> /COL11
- J1 pad 9: /COL3 -> /COL10
- J2 pad 11: /COL11 -> /COL4
- J2 pad 13: /COL12 -> /COL5
- J2 pad 14: /COL13 -> /COL6
- J2 pad 3: /COL7 -> /COL0
- J2 pad 5: /COL8 -> /COL1
- J2 pad 7: /COL9 -> /COL2
- J2 pad 9: /COL10 -> /COL3
- U1 pad 1: /COL0 -> /COL13
- U1 pad 10: /COL5 -> /COL8
- U1 pad 11: /COL6 -> /COL7
- U1 pad 2: /COL1 -> /COL12
- U1 pad 21: /COL13 -> /COL6
- U1 pad 22: /COL12 -> /COL5
- U1 pad 24: /COL11 -> /COL4
- U1 pad 25: /COL10 -> /COL3
- U1 pad 26: /COL9 -> /COL2
- U1 pad 27: /COL8 -> /COL1
- U1 pad 29: /COL7 -> /COL0
- U1 pad 4: /COL2 -> /COL11
- U1 pad 5: /COL3 -> /COL10
- U1 pad 9: /COL4 -> /COL9
Routing:
- net /COL1: track 36.1 -> 14.4 mm
- net /COL0: track 35.0 -> 13.4 mm
- net /COL12: track 16.5 -> 36.1 mm
- net /COL3: track 33.7 -> 14.4 mm
- net /COL10: track 14.4 -> 33.7 mm
- net /COL2: track 32.5 -> 14.4 mm
- net /COL11: track 14.4 -> 32.5 mm
- net /COL13: track 19.1 -> 35.0 mm
- net /COL8: track 14.4 -> 25.2 mm
- net /COL9: track 14.4 -> 25.0 mm
- net /COL4: track 25.0 -> 14.4 mm
- net /COL5: track 25.2 -> 16.5 mm
- net /COL7: track 13.4 -> 21.6 mm
- net /COL6: track 21.6 -> 19.1 mm
